Commit message: Simplify the hokuyo attachment to a fixed link
A fixed joint seems to work just fine here, and eliminates the need for a motor
to hold the hokuyo still.

This makes it much easier to use a robot_state_publisher in future.

File: racecar_description/urdf/macros.xacro (robot description, xacro)
@@ -117,15 +117,3 @@
   </transmission>
 </xacro:macro>
-<xacro:macro name="hokuyo_transmission" params="name">
-  <transmission name="${name}_transmission" type="SimpleTransmission">
-    <type>transmission_interface/SimpleTransmission</type>
-    <joint name="${name}_joint">
-      <hardwareInterface>EffortJointInterface</hardwareInterface>
-    </joint>
-    <actuator name="${name}_motor">
-      <hardwareInterface>EffortJointInterface</hardwareInterface>
-      <mechanicalReduction>1</mechanicalReduction>
-    </actuator>
-  </transmission>
-</xacro:macro>
 </robot>

File: racecar_description/urdf/racecar.xacro (robot description, xacro)
@@ -158,12 +158,10 @@
     </visual>
   </link>
-  <joint name="hokuyo_joint" type="revolute">
+  <joint name="hokuyo_joint" type="fixed">
     <origin xyz="0.325 0.0 0.065" rpy="0 0 0"/>
     <parent link="chassis" />
     <child link="hokuyo_link" />
     <axis xyz="0 0 1" />
-    <limit lower="0.0" upper="0.0" effort="0.0" velocity="0.0" />
   </joint>
-  <xacro:hokuyo_transmission name="hokuyo" />
   <!-- Add the remaining xacros -->
   <xacro:include filename="$(find racecar_description)/urdf/racecar.gazebo" />
