Commit message: Actually fix the steering direction

File: racecar_description/urdf/racecar.xacro (robot description, xacro)
@@ -75,5 +75,5 @@
     <parent link="chassis" />
     <child link="left_steering_hinge" />
-    <axis xyz="1 0 0" />
+    <axis xyz="-1 0 0" />
     <limit lower="-1.0" upper="1.0" effort="10" velocity="100" />
   </joint>
@@ -93,5 +93,5 @@
     <parent link="chassis" />
     <child link="right_steering_hinge" />
-    <axis xyz="1 0 0" />
+    <axis xyz="-1 0 0" />
     <limit lower="-1.0" upper="1.0" effort="10" velocity="100" />
   </joint>

Commit message: Add the left zed rgb camera to the simulator
This should correctly handle:
* The image topic, at 30Hz VGA
* The camera_info topic
* The tf frame name, maybe. There could be an issue with optical vs true frame,
  as described at http://www.ros.org/reps/rep-0103.html#suffix-frames. At any
  rate, it describes the tf referenced by the zed_tf launch file, allowing a
  robot_state_publisher node to be used in future
* Sort of looking like the zed

Co-authored by Ernie Ho, @g41903

File: racecar_description/urdf/racecar.xacro (robot description, xacro)
@@ -166,4 +166,60 @@
   </joint>
   <xacro:hokuyo_transmission name="hokuyo" />
+  <!-- zed camera -->
+  <link name="zed_camera_link">
+    <inertial>
+      <mass value="1e-5" />
+      <origin xyz="0 0 0" rpy="0 0 0"/>
+      <inertia ixx="1e-6" ixy="0" ixz="0" iyy="1e-6" iyz="0" izz="1e-6" />
+    </inertial>
+    <collision>
+      <origin xyz="0 0 0" rpy="0 0 0"/>
+      <geometry>
+        <box size="0.033 0.175 0.030"/>
+      </geometry>
+    </collision>
+    <visual>
+      <origin xyz="0 0 0" rpy="0 0 0"/>
+      <geometry>
+        <box size="0.033 0.175 0.030"/>
+      </geometry>
+      <material name="red"/>
+    </visual>
+  </link>
+  <joint name="zed_camera_joint" type="fixed">
+    <origin xyz="0.390 0 0.04" rpy="0 0 0"/>
+    <parent link="chassis"/>
+    <child link="zed_camera_link"/>
+    <axis xyz="0 0 1" />
+    <!-- <limit lower="0.0" upper="0.0" effort="0.0" velocity="0.0" /> -->
+  </joint>
+  <!-- zed camera lenses -->
+  <!-- It seems these have to have a non-zero mass to have a camera attached? -->
+  <link name="camera_link"><!-- this needs to match the name in zed_wrapper/zed_tf.launch -->
+    <inertial>
+      <mass value="1e-5" />
+      <origin xyz="0 0 0" rpy="0 0 0"/>
+      <inertia ixx="1e-6" ixy="0" ixz="0" iyy="1e-6" iyz="0" izz="1e-6" />
+    </inertial>
+  </link>
+  <link name="zed_camera_right_link">
+    <inertial>
+      <mass value="1e-5" />
+      <origin xyz="0 0 0" rpy="0 0 0"/>
+      <inertia ixx="1e-6" ixy="0" ixz="0" iyy="1e-6" iyz="0" izz="1e-6" />
+    </inertial>
+  </link>
+  <joint name="zed_camera_left_joint" type="fixed">
+    <origin xyz="0 0.06 0" rpy="0 0 0"/>
+    <parent link="zed_camera_link"/>
+    <child link="camera_link"/>
+    <axis xyz="0 0 1" />
+  </joint>
+  <joint name="zed_camera_right_joint" type="fixed">
+    <origin xyz="0 -0.06 0" rpy="0 0 0"/>
+    <parent link="zed_camera_link"/>
+    <child link="zed_camera_right_link"/>
+    <axis xyz="0 0 1" />
+  </joint>
   <!-- Add the remaining xacros -->
   <xacro:include filename="$(find racecar_description)/urdf/racecar.gazebo" />

Commit message: Add a base_link frame, which ros expects to exist

File: racecar_description/urdf/racecar.xacro (robot description, xacro)
@@ -3,4 +3,5 @@
   <xacro:include filename="$(find racecar_description)/urdf/macros.xacro" />
   <!-- Add chassis and it's inertia link -->
+  <link name="base_link" />
   <link name="chassis">
     <visual>
@@ -9,4 +10,9 @@
     </visual>
   </link>
+  <joint name="base_link_joint" type="fixed">
+    <origin xyz="0 0 0" rpy="0 0 0" />
+    <parent link="base_link" />
+    <child link="chassis" />
+  </joint>
   <link name="chassis_inertia">
     <inertial>

Commit message: Rename the laser frame to be the same as in the hardware

File: racecar_description/urdf/racecar.xacro (robot description, xacro)
@@ -146,5 +146,5 @@
   <xacro:wheel_transmission name="right_front_wheel" />
   <!-- Add Hokuyo laser scanner -->
-  <link name="hokuyo_link">
+  <link name="laser">
     <inertial>
       <xacro:hokuyo_inertial_params />
@@ -167,5 +167,5 @@
     <origin xyz="0.325 0.0 0.065" rpy="0 0 0"/>
     <parent link="chassis" />
-    <child link="hokuyo_link" />
+    <child link="laser" />
     <axis xyz="0 0 1" />
     <limit lower="0.0" upper="0.0" effort="0.0" velocity="0.0" />

Commit message: Correct laser to base_link frame
Car no longer intersects the ground

File: racecar_description/urdf/racecar.xacro (robot description, xacro)
@@ -11,5 +11,5 @@
   </link>
   <joint name="base_link_joint" type="fixed">
-    <origin xyz="0 0 0" rpy="0 0 0" />
+    <origin xyz="0 0 0.05" rpy="0 0 0" />
     <parent link="base_link" />
     <child link="chassis" />
@@ -165,5 +165,5 @@
   </link>
   <joint name="hokuyo_joint" type="fixed">
-    <origin xyz="0.325 0.0 0.065" rpy="0 0 0"/>
+    <origin xyz="0.265 0.0 0.075" rpy="0 0 0"/>
     <parent link="chassis" />
     <child link="laser" />
